File: Arduino_codec.kicad_pcb (KiCad board)
At the start: 4 copper layers, 58.4 x 99.1 mm, 118 parts, among them J1 Screw_Terminal_01x02, J10 Screw_Terminal_01x02, J2 Screw_Terminal_01x03, J3 Conn_02x08_Odd_Even, J4 Conn_02x10_Odd_Even, J5 Conn_02x15_Odd_Even, J6 Conn_02x17_Odd_Even, J7 Screw_Terminal_01x02, J8 Screw_Terminal_01x02, J9 Screw_Terminal_01x02, Q1 MMBT4401L, Q2 MMBT4403LT1G, Q3 MMBT4401L, Q4 MMBT4401L, U1 TPSM84203, U2 TPSM84205, U3 NE5532, U4 LP2985IM5-5.0/NOPB, U5 PCM1793DBR, U6 PCM1802

Commit message: 1st review before fabrication
Ready to review before fabrication outputs.
Parts:
- removed C10, C8: 220uF, Capacitor_THT:CP_Radial_D8.0mm_P3.50mm
- removed C11, C16, C9: 10nF, Capacitor_SMD:C_0603_1608Metric_Pad1.05x0.95mm_HandSolder
- removed C12: 10uF, Capacitor_Tantalum_SMD:CP_EIA-6032-20_AVX-F_Pad2.25x2.35mm_HandSolder
- removed C13: 22nF, Capacitor_SMD:C_0603_1608Metric_Pad1.05x0.95mm_HandSolder
- removed C15: 100uF, Capacitor_Tantalum_SMD:CP_EIA-7343-30_AVX-N_Pad2.25x2.55mm_HandSolder
- removed C7: 470uF, Capacitor_THT:CP_Radial_D8.0mm_P3.50mm
- removed D1, D2: US1D, Diode_SMD:D_SMA
- removed D10, D11, D7, D9: LED, LED_SMD:LED_0603_1608Metric_Pad1.05x0.95mm_HandSolder
- removed Q1: MMBT4401L, Package_TO_SOT_SMD:SOT-23
- removed Q2: MMBT4403LT1G, Package_TO_SOT_SMD:SOT-23
- removed R35, R39: 3.3K, Resistor_SMD:R_0603_1608Metric_Pad1.05x0.95mm_HandSolder
- removed R37: 1K, Resistor_SMD:R_0603_1608Metric_Pad1.05x0.95mm_HandSolder
- removed R38: 270, Resistor_SMD:R_0603_1608Metric_Pad1.05x0.95mm_HandSolder
- C1: value 10nF -> 10uF; footprint Capacitor_SMD:C_0603_1608Metric_Pad1.05x0.95mm_HandSolder -> Capacitor_Tantalum_SMD:CP_EIA-6032-20_AVX-F_Pad2.25x2.35mm_HandSolder
- C2, C5: footprint Capacitor_SMD:C_0603_1608Metric_Pad1.05x0.95mm_HandSolder -> Capacitor_SMD:C_0603_1608Metric_Pad1.08x0.95mm_HandSolder
- C3: value 470uF -> 10nF; footprint Capacitor_THT:CP_Radial_D8.0mm_P3.50mm -> Capacitor_SMD:C_0603_1608Metric_Pad1.08x0.95mm_HandSolder
- C6: value 10nF -> 100uF; footprint Capacitor_SMD:C_0603_1608Metric_Pad1.05x0.95mm_HandSolder -> Capacitor_Tantalum_SMD:CP_EIA-7343-30_AVX-N_Pad2.25x2.55mm_HandSolder
- J1: value Screw_Terminal_01x02 -> Conn_01x02; footprint Arduino_codec:TerminalBlock_Phoenix_MPT-0,5-2-2.54_1x02_P2.54mm_Horizontal -> Connector_PinHeader_2.54mm:PinHeader_1x02_P2.54mm_Vertical
- NT1: moved to B.Cu
- R1, R2: value 560 -> 270; footprint Resistor_SMD:R_0603_1608Metric_Pad1.05x0.95mm_HandSolder -> Resistor_SMD:R_0603_1608Metric_Pad0.98x0.95mm_HandSolder
- R33, R34: value 8.2K -> 2.7K
- U1: value TPSM84203 -> LDS3985M33R; footprint Package_TO_SOT_THT:TO-220-3_Vertical -> Package_TO_SOT_SMD:SOT-23-5_HandSoldering
- moved J2 97.0 mm to (163.2, 142.2), turned to 0 degrees
- moved C22 54.1 mm to (144.5, 120.7), turned to -90 degrees
- moved C23 52.1 mm to (147.6, 120.9), turned to -90 degrees
- moved C24 50.9 mm to (156.2, 120.7)
- moved C4 48.0 mm to (157.2, 93.2)
- moved C1 47.4 mm to (143.5, 94.0), turned to 90 degrees
- moved C26 47.1 mm to (153.0, 121.3)
- moved U4 47.1 mm to (150.4, 119.6)
- moved C25 46.7 mm to (150.5, 123.8), turned to 180 degrees
- moved D6 44.8 mm to (150.4, 82.5)
- moved C3 44.8 mm to (150.5, 95.9), turned to 180 degrees
- moved D5 44.2 mm to (157.5, 82.5)
- moved Q3 44.1 mm to (157.5, 79.0)
- moved C2 42.2 mm to (146.7, 93.6), turned to 90 degrees
- moved Q4 41.5 mm to (150.4, 79.0)
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Connections:
- net /~ADC_PWDN renamed /~{ADC_PWDN}
- net /~DAC_RST renamed /~{DAC_RST}
- C1 pad 1: +VDC -> +5VD
- C1 pad 2: Net-(C1-Pad2) -> GND
- C14 pad 1: +VDC -> VCC
- C14 pad 2: GND -> AGND
- C17 pad 1: +VDC -> VCC
- C17 pad 2: GND -> AGND
- C18 pad 1: VDDA -> VCC
- C19 pad 1: VDDA -> VCC
- C2 pad 1: +VDC -> +5VD
- C20 pad 2: VSSA -> VSS
- C21 pad 2: VSSA -> VSS
- C24 pad 1: VDDA -> VCC
- C25 pad 1: VDDA -> VCC
- C3 pad 1: +VDC -> Net-(C3-Pad1)
- C39 pad 1: /Vin_L -> /Vin_R
- C4 pad 1: +VDC -> +3V3
- C4 pad 2: -VDC -> GND
- C40 pad 1: /Vin_R -> /Vin_L
- C48 pad 1: +5VD -> +5V
- C49 pad 1: +5VD -> +5V
- C5 pad 1: -VDC -> +3V3
- C5 pad 2: Net-(C1-Pad2) -> GND
- C6 pad 1: GND -> +5VD
- C6 pad 2: -VDC -> GND
- D5 pad 2: +3V3 -> Net-(D5-Pad2)
- D6 pad 2: +3V3 -> Net-(D6-Pad2)
- J1 pad 1: Net-(C1-Pad2) -> +5VD
- J1 pad 2: GND -> +5V
- J2 pad 1: +VDC -> VCC
- J2 pad 2: GND -> AGND
- J2 pad 3: -VDC -> VSS
- J3 pad 1: Net-(J3-Pad1) -> unconnected-(J3-Pad1)
- J3 pad 15: Net-(J3-Pad15) -> unconnected-(J3-Pad15)
- J3 pad 5: Net-(J3-Pad5) -> unconnected-(J3-Pad5)
- J3 pad 7: Net-(J3-Pad7) -> unconnected-(J3-Pad7)
- J4 pad 6: Net-(J4-Pad6) -> unconnected-(J4-Pad6)
- J5 pad 13: Net-(J5-Pad13) -> unconnected-(J5-Pad13)
- J5 pad 15: Net-(J5-Pad15) -> unconnected-(J5-Pad15)
- J6 pad 1: Net-(J6-Pad1) -> unconnected-(J6-Pad1)
- J6 pad 21: Net-(J6-Pad21) -> unconnected-(J6-Pad21)
- J6 pad 25: Net-(J6-Pad25) -> unconnected-(J6-Pad25)
- J6 pad 29: Net-(J6-Pad29) -> unconnected-(J6-Pad29)
- J6 pad 31: Net-(J6-Pad31) -> unconnected-(J6-Pad31)
- J6 pad 33: Net-(J6-Pad33) -> unconnected-(J6-Pad33)
- R1 pad 1: Net-(C8-Pad1) -> Net-(D5-Pad2)
- R1 pad 2: +VDC -> +3V3
- R2 pad 1: -VDC -> Net-(D6-Pad2)
- R2 pad 2: Net-(C10-Pad2) -> +3V3
- U1 pad 1: +VDC -> +5VD
- U1 pad 3: +3V3 -> +5VD
- U2 pad 1: +VDC -> VCC
- U2 pad 2: GND -> AGND
- U2 pad 3: +5VD -> +5V
- U3 pad 4: VSSA -> VSS
- U3 pad 8: VDDA -> VCC
- U4 pad 1: VDDA -> VCC
- U4 pad 3: VDDA -> VCC
Routing:
- net VCC: track 0.00 -> 141.8 mm, vias 0 -> 7
- net +3V3: track 194.9 -> 59.2 mm, vias 9 -> 12
- net AGND: track 70.3 -> 201.9 mm, vias 25 -> 22
- net +VDC: track 113.6 -> 0.00 mm, vias 3 -> 0
- net VDDA: track 103.9 -> 0.00 mm, vias 2 -> 0
- net VSSA: track 96.4 -> 0.00 mm, vias 3 -> 0
- net +5VA: track 126.3 -> 44.5 mm, vias 4 -> 5
- net -VDC: track 76.2 -> 0.00 mm, vias 2 -> 0
- net Net-(R34-Pad1): track 2.60 -> 32.0 mm, vias 0 -> 2
- net Net-(R33-Pad1): track 4.52 -> 31.7 mm, vias 0 -> 2
- net Net-(C39-Pad2): track 9.79 -> 34.2 mm, vias 0 -> 1
- net VSS: track 0.00 -> 24.0 mm, vias 0 -> 3
- net Net-(C1-Pad2): track 19.4 -> 0.00 mm
- net Net-(C40-Pad2): track 14.1 -> 33.0 mm, vias 0 -> 1
- net /ADC_BCK: track 37.0 -> 55.3 mm, vias 1 -> 2
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- added copper zone on In2.Cu, net +3V3
- added copper zone on In1.Cu, net +5VA
- added copper zone on In2.Cu, net +5VA
- added copper zone on In1.Cu, net +5VD
- added copper zone on B.Cu, net AGND
- added copper zone on F.Cu, net AGND
- added copper zone on In1.Cu, net VCC
- added copper zone on In2.Cu, net VSS
- removed copper zone on In1.Cu, net AGND
- removed copper zone on In2.Cu, net GND
Other:
- board size 58.4 x 99.1 mm -> 58.4 x 85.7 mm
- net class Default removed
- board text added: "Audio ADC / DAC for STM32 Nucleo Alberto Fahrenkrog 2022"
- board text removed: "+V"
- board text removed: "-V"
- board text removed: "3V3"
- board text removed: "5VA"
- board text removed: "Audio ADC / DAC for STM32 Nucleo Alberto Fahrenkrog 2021"
- board text removed: "V AC In (9V)"
