File: Arduino_codec.sch (KiCad schematic (older format))
At the start: 118 parts, among them J1 Screw_Terminal_01x02, J10 Screw_Terminal_01x02, J2 Screw_Terminal_01x03, J3 Conn_02x08_Odd_Even, J4 Conn_02x10_Odd_Even, J5 Conn_02x15_Odd_Even, J6 Conn_02x17_Odd_Even, J7 Screw_Terminal_01x02, J8 Screw_Terminal_01x02, J9 Screw_Terminal_01x02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

Commit message: 1st review before fabrication
Ready to review before fabrication outputs.
Parts:
- removed C1, C11, C16, C6, C9: 10nF, Capacitor_SMD:C_0603_1608Metric_Pad1.05x0.95mm_HandSolder, symbol Device:C
- removed C10, C8: 220uF, Capacitor_THT:CP_Radial_D8.0mm_P3.50mm, symbol Device:CP
- removed C12: 10uF, Capacitor_Tantalum_SMD:CP_EIA-6032-20_AVX-F_Pad2.25x2.35mm_HandSolder, symbol Device:CP
- removed C13: 22nF, Capacitor_SMD:C_0603_1608Metric_Pad1.05x0.95mm_HandSolder, symbol Device:C
- removed C15: 100uF, Capacitor_Tantalum_SMD:CP_EIA-7343-30_AVX-N_Pad2.25x2.55mm_HandSolder, symbol Device:CP
- removed C3, C7: 470uF, Capacitor_THT:CP_Radial_D8.0mm_P3.50mm, symbol Device:CP
- removed C4: 10uF, Capacitor_Tantalum_SMD:CP_EIA-6032-20_AVX-F_Pad2.25x2.35mm_HandSolder, symbol Device:C
- removed D1, D2: US1D, Diode_SMD:D_SMA, symbol Diode:US1D
- removed D11, D7: LED, LED_SMD:LED_0603_1608Metric_Pad1.05x0.95mm_HandSolder, symbol Device:LED
- removed J1: Screw_Terminal_01x02, Arduino_codec:TerminalBlock_Phoenix_MPT-0,5-2-2.54_1x02_P2.54mm_Horizontal, symbol Connector:Screw_Terminal_01x02
- removed Q1: MMBT4401L, Package_TO_SOT_SMD:SOT-23, symbol Device:Q_NPN_BEC
- removed Q2: MMBT4403LT1G, Package_TO_SOT_SMD:SOT-23, symbol Device:Q_PNP_BEC
- removed R1, R2: 560, Resistor_SMD:R_0603_1608Metric_Pad1.05x0.95mm_HandSolder, symbol Device:R_Small_US
- removed R35, R39: 3.3K, Resistor_SMD:R_0603_1608Metric_Pad1.05x0.95mm_HandSolder, symbol Device:R_Small_US
- removed U1: TPSM84203, Package_TO_SOT_THT:TO-220-3_Vertical, symbol Arduino_codec-rescue:TPSM84203-Arduino_codec
- added C1, C4: 10uF, Capacitor_Tantalum_SMD:CP_EIA-6032-20_AVX-F_Pad2.25x2.35mm_HandSolder, symbol Device:CP
- added C3: 10nF, Capacitor_SMD:C_0603_1608Metric_Pad1.08x0.95mm_HandSolder, symbol Device:C
- added U1: LDS3985M33R, Package_TO_SOT_SMD:SOT-23-5_HandSoldering, symbol Regulator_Linear:LP2985-5.0
- C2, C5: footprint Capacitor_SMD:C_0603_1608Metric_Pad1.05x0.95mm_HandSolder -> Capacitor_SMD:C_0603_1608Metric_Pad1.08x0.95mm_HandSolder
Connections:
- net labels added: VCC, VSS
- net labels removed: +VDC, -VDC, VDDA, VSSA
- wire segments 445 -> 403
Other:
- moved on the sheet: C17, C23, C25, C26, C34, C36, C38, C39, C40, C42, C49, D10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
