File: Arduino_codec.kicad_sch (KiCad schematic)
At the start: 97 parts, among them J1 Conn_01x02, J10 Screw_Terminal_01x02, J2 Screw_Terminal_01x03, J3 Conn_02x08_Odd_Even, J4 Conn_02x10_Odd_Even, J5 Conn_02x15_Odd_Even, J6 Conn_02x17_Odd_Even, J7 Screw_Terminal_01x02, J8 Screw_Terminal_01x02, J9 Screw_Terminal_01x02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

Commit message: Simplified branch
Parts:
- removed C14: 10uF, Capacitor_Tantalum_SMD:CP_EIA-6032-20_AVX-F_Pad2.25x2.35mm_HandSolder, symbol Device:CP
- removed C17: 10nF, Capacitor_SMD:C_0603_1608Metric_Pad1.05x0.95mm_HandSolder, symbol Device:C
- removed C48, C6: 100uF, Capacitor_Tantalum_SMD:CP_EIA-7343-30_AVX-N_Pad2.25x2.55mm_HandSolder, symbol Device:CP
- removed C49: 22nF, Capacitor_SMD:C_0603_1608Metric_Pad1.05x0.95mm_HandSolder, symbol Device:C
- removed J1: Conn_01x02, Connector_PinHeader_2.54mm:PinHeader_1x02_P2.54mm_Vertical, symbol Connector_Generic:Conn_01x02
- removed J3: Conn_02x08_Odd_Even, Connector_PinHeader_2.54mm:PinHeader_2x08_P2.54mm_Vertical, symbol Connector_Generic:Conn_02x08_Odd_Even
- removed J5: Conn_02x15_Odd_Even, Connector_PinHeader_2.54mm:PinHeader_2x15_P2.54mm_Vertical, symbol Connector_Generic:Conn_02x15_Odd_Even
- removed J6: Conn_02x17_Odd_Even, Connector_PinHeader_2.54mm:PinHeader_2x17_P2.54mm_Vertical, symbol Connector_Generic:Conn_02x17_Odd_Even
- removed U2: TPSM84205, Package_TO_SOT_THT:TO-220-3_Vertical, symbol Arduino_codec-rescue:TPSM84205-Arduino_codec
- added FB1: FerriteBead, symbol Device:FerriteBead
- added J1: Conn_02x10_Odd_Even, Connector_PinHeader_2.54mm:PinHeader_2x10_P2.54mm_Vertical, symbol Connector_Generic:Conn_02x10_Odd_Even
Connections:
- net PA4 is gone; now on net DEMP0: J4.17 (Pin_17)
- net PA5 is gone; now on net +3V3: J4.10 (Pin_10)
- net PA6 is gone; now on net GND: J4.12 (Pin_12)
- net PA7 is gone; now on net GND: J4.14 (Pin_14)
- net PB13 is gone; now on net DAC_WS: J4.5 (Pin_5)
- net PB4 is gone; now on net ~{DAC_RST}: J4.19 (Pin_19)
- net PB8 is gone; now on net MUTE: J4.2 (Pin_2)
- net PB9 is gone; now on net +3V3: J4.4 (Pin_4)
- net PD14 is gone; now on net GND: J4.16 (Pin_16)
- net PD15 is gone; now on net GND: J4.18 (Pin_18)
- net PF12 is gone; now on net GND: J4.20 (Pin_20)
- net +3V3: now also J4.6 (Pin_6), J4.8 (Pin_8), J1.10 (Pin_10), J1.12 (Pin_12), J1.6 (Pin_6), J1.8 (Pin_8)
- net +5VA: now also R36.2, FB1.2; no longer C22.1, C23.1, U4.5 (VOUT)
- net +5VD: now also C22.1, C23.1, U4.5 (VOUT), FB1.1; no longer R36.2
- net ADC_BCK: now also J1.3 (Pin_3)
- net ADC_FMT0: now also J1.11 (Pin_11)
- net ADC_FMT1: now also J1.9 (Pin_9)
- net ADC_MCK: now also J1.1 (Pin_1); no longer J4.1 (Pin_1)
- net ADC_SD: now also J1.7 (Pin_7); no longer J4.3 (Pin_3)
- net ADC_WS: now also J1.5 (Pin_5); no longer J4.7 (Pin_7)
- net BYPAS: now also J1.17 (Pin_17)
- net DAC_BCK: now also J4.3 (Pin_3); no longer J4.15 (Pin_15)
- net DAC_FMT0: now also J4.13 (Pin_13)
- net DAC_FMT1: now also J4.11 (Pin_11)
- net DAC_FMT2: now also J4.9 (Pin_9)
- net DAC_MCK: now also J4.1 (Pin_1); no longer J4.11 (Pin_11)
- net DAC_SD: now also J4.7 (Pin_7); no longer J4.13 (Pin_13)
- net DAC_WS: no longer J4.9 (Pin_9)
- net DEMP1: now also J4.15 (Pin_15)
- net FSYNC: now also J1.4 (Pin_4)
- net GND: now also J1.14 (Pin_14), J1.16 (Pin_16), J1.18 (Pin_18), J1.20 (Pin_20); no longer J4.8 (Pin_8)
- net MODE0: now also J1.15 (Pin_15)
- net MODE1: now also J1.13 (Pin_13)
- net OSR: now also J1.2 (Pin_2)
- net ~{ADC_PWDN}: now also J1.19 (Pin_19)
- no-connect marks 66 -> 0
Other:
- note removed: "(3V3 Ext)"
- note removed: "(AVDD)"
- note removed: "(PA0)"
- note removed: "(PA15)"
- note removed: "(PA7)"
- note removed: "(PB0)"
- note removed: "(PB1)"
- note removed: "(PB10)"
- note removed: "(PB12)"
- note removed: "(PB13)"
- note removed: "(PB15)"
- note removed: "(PB2)"
- note removed: "(PB3)"
- note removed: "(PB5)"
- note removed: "(PB6)"
- note removed: "(PC2)"
- note removed: "(PC6)"
- note removed: "(PC7)"
- note removed: "(PD11)"
- note removed: "(PD12)"
- note removed: "(PD13)"
- note removed: "(PD3)"
- note removed: "(PD4)"
- note removed: "(PD5)"
- note removed: "(PD6)"
- note removed: "(PD7)"
- note removed: "(PE0)"
- note removed: "(PE2)"
- note removed: "(PE3)"
- note removed: "(PE4)"
- note removed: "(PE5)"
- note removed: "(PE6)"
- note removed: "(PF4)"
- note removed: "(PF7)"
- note removed: "(PF8)"
- note removed: "(PF9)"
- note removed: "(PG1)"
- note removed: "(RESET)"
- moved on the sheet: C1, C2, C3, C4, C5, D8, J4, R36, U1
